File: PCB/POV display.kicad_pcb (KiCad board)
At the start: 2 copper layers, 151.9 x 141.8 mm, 120 parts, among them J1 Conn_01x04_Pin, J2 USB_C_Receptacle_USB2.0_16P, J3 Conn_01x04_Pin, J4 USB_C_Receptacle_USB2.0_16P, Q1 HL6042, U1 RP2354A, U2 SC7A20, U3 1.1V @ 300mA, U4 74HC595D, U5 74HC595D, U6 CH572D, U7 AMS1117, X1 X322512MSB4SI, X2 Y201632MFBCX

Commit message: firmware initial complete
Parts:
- removed TP1, TP2: TestPoint, TestPoint:TestPoint_Pad_D1.0mm
- added AE1: Antenna_Chip, Capacitor_SMD:C_1206_3216Metric, F.Cu at (100.1, 124.8)
- added C24: 100nF, PCM_JLCPCB:C_0402, F.Cu at (133.2, 136.2)
- added C25: 100nF, PCM_JLCPCB:C_0402, F.Cu at (124.9, 141.3)
- added C26: 100nF, PCM_JLCPCB:C_0402, F.Cu at (131.0, 140.8)
- added C5: 100nF, PCM_JLCPCB:C_0402, F.Cu at (120.9, 136.0)
- added TP13: TestPoint, TestPoint:TestPoint_Pad_D1.0mm, F.Cu at (122.9, 125.3)
- added TP14: TestPoint, TestPoint:TestPoint_Pad_D1.0mm, F.Cu at (122.8, 123.2)
- J1, J3: moved to B.Cu
- moved R51 161.9 mm to (119.0, 130.4), turned to 180 degrees
- moved R52 161.9 mm to (119.0, 132.2), turned to 180 degrees
- moved R54 95.0 mm to (114.7, 124.6), turned to -90 degrees
- moved R55 95.0 mm to (113.2, 124.6), turned to -90 degrees
- moved S1 91.9 mm to (135.5, 151.5), turned to 90 degrees
- moved Q1 91.3 mm to (113.4, 113.5)
- moved C22 90.5 mm to (107.5, 113.2)
- moved C23 90.5 mm to (111.7, 119.0)
- moved D17 90.5 mm to (106.6, 110.9)
- moved U7 90.5 mm to (105.8, 118.0)
- moved R48 90.5 mm to (112.1, 109.7)
- moved R32 85.2 mm to (135.4, 146.7), turned to 90 degrees
- moved R38 77.2 mm to (109.1, 145.2)
- moved R34 77.2 mm to (110.6, 145.2)
- moved TP8 77.0 mm to (100.7, 132.8)
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Connections:
- R15 pad 1: Net-(U1-GPIO2) -> Net-(U1-GPIO22)
- R16 pad 1: Net-(U1-GPIO3) -> Net-(U1-GPIO19)
- R17 pad 1: Net-(U1-GPIO5) -> Net-(U1-GPIO25)
- R51 pad 1: Net-(U1-GPIO8) -> Net-(U1-GPIO21)
- R51 pad 2: unconnected-(R51-Pad2) -> /INT2
- R52 pad 1: Net-(U1-GPIO7) -> Net-(U1-GPIO23)
- R52 pad 2: unconnected-(R52-Pad2) -> /INT1
- R8 pad 1: Net-(U1-GPIO0) -> Net-(U1-GPIO20)
- R9 pad 1: Net-(U1-GPIO1) -> Net-(U1-GPIO24)
- U1 pad 10: Net-(U1-GPIO7) -> /GND_LED11
- U1 pad 12: Net-(U1-GPIO8) -> /GND_LED10
- U1 pad 13: unconnected-(U1-GPIO9-Pad13) -> /GND_LED9
- U1 pad 14: /GND_LED0 -> /GND_LED8
- U1 pad 15: /GND_LED1 -> /GND_LED7
- U1 pad 16: /GND_LED2 -> /GND_LED6
- U1 pad 17: /GND_LED3 -> /GND_LED5
- U1 pad 19: /GND_LED5 -> /GND_LED3
- U1 pad 2: Net-(U1-GPIO0) -> unconnected-(U1-GPIO0-Pad2)
- U1 pad 24: unconnected-(U1-SWCLK-Pad24) -> Net-(U1-SWCLK)
- U1 pad 25: unconnected-(U1-SWDIO-Pad25) -> Net-(U1-SWDIO)
- U1 pad 27: /GND_LED6 -> /GND_LED2
- U1 pad 28: /GND_LED7 -> /GND_LED1
- U1 pad 29: /GND_LED8 -> /GND_LED0
- U1 pad 3: Net-(U1-GPIO1) -> unconnected-(U1-GPIO1-Pad3)
- U1 pad 31: /GND_LED9 -> Net-(U1-GPIO19)
- U1 pad 32: /GND_LED10 -> Net-(U1-GPIO20)
- U1 pad 33: /GND_LED11 -> Net-(U1-GPIO21)
- U1 pad 34: /GND_LED12 -> Net-(U1-GPIO22)
- U1 pad 35: /GND_LED13 -> Net-(U1-GPIO23)
- U1 pad 36: /GND_LED14 -> Net-(U1-GPIO24)
- U1 pad 37: /GND_LED15 -> Net-(U1-GPIO25)
- U1 pad 4: Net-(U1-GPIO2) -> unconnected-(U1-GPIO2-Pad4)
- U1 pad 5: Net-(U1-GPIO3) -> /GND_LED15
- U1 pad 7: unconnected-(U1-GPIO4-Pad7) -> /GND_LED14
- U1 pad 8: Net-(U1-GPIO5) -> /GND_LED13
- U1 pad 9: unconnected-(U1-GPIO6-Pad9) -> /GND_LED12
- U6 pad 21: (no net) -> GND
Routing:
- net /CS_ACC: track 0.00 -> 130.6 mm, vias 0 -> 3
- net /INT1: track 0.00 -> 127.4 mm, vias 0 -> 2
- net /INT2: track 0.00 -> 124.5 mm, vias 0 -> 3
- net /SCK: track 0.00 -> 121.2 mm, vias 0 -> 4
- net /MISO: track 0.00 -> 120.3 mm, vias 0 -> 2
- net /MOSI: track 0.00 -> 117.0 mm
- net /GND_LED15: track 0.00 -> 109.7 mm
- net +3V3_RPI: track 0.00 -> 104.0 mm, vias 0 -> 10
- net /CS_SR: track 0.00 -> 103.6 mm, vias 0 -> 4
- net /GND_LED14: track 0.00 -> 103.2 mm
- net /GND_LED13: track 0.00 -> 98.2 mm
- net /GND_LED12: track 0.00 -> 93.2 mm
- net /GND_LED11: track 0.00 -> 88.2 mm
- net VBAT: track 0.00 -> 84.2 mm, vias 0 -> 2
- net /GND_LED10: track 0.00 -> 81.5 mm
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- added copper zone on In2.Cu, net +3V3
- added copper zone on B.Cu, net GND
- added copper zone on F.Cu, net GND
- added copper zone on In1.Cu, net GND
Other:
- board size 151.9 x 141.8 mm -> 41.2 x 129 mm
- copper layers 2 -> 4
